Commit message: working launch file and urdf including ros control for arm; cautionary WIP save

File: description/robots/youbot_arm_only.urdf.xacro (robot description, xacro)
@@ -7,13 +7,13 @@
   <!-- The following included files set up definitions of parts of the robot body -->
   <!-- misc common stuff? -->
-  <xacro:include filename="$(find youbot_description)/urdf/common.xacro" />
+  <xacro:include filename="$(find youbot_ros2)/description/urdf/common.xacro" />
   <!-- materials for visualization -->
-  <xacro:include filename="$(find youbot_description)/urdf/materials.urdf.xacro" />
+  <xacro:include filename="$(find youbot_ros2)/description/urdf/materials.urdf.xacro" />
   <!-- youbot arm -->
-  <xacro:include filename="$(find youbot_description)/urdf/youbot_arm/arm.urdf.xacro" />
+  <xacro:include filename="$(find youbot_ros2)/description/urdf/youbot_arm/arm.urdf.xacro" />
   <!-- youbot arm -->
-  <xacro:include filename="$(find youbot_description)/urdf/youbot_gripper/gripper.urdf.xacro" />
+  <!-- <xacro:include filename="$(find youbot_ros2)/description/urdf/youbot_gripper/gripper.urdf.xacro" /> -->
   <!-- controller manager -->
-  <!-- <xacro:include filename="$(find youbot_description)/controller/ros_controller.urdf.xacro" /> -->
+  <xacro:include filename="$(find youbot_ros2)/control/arm.control.urdf.xacro" />
   <!-- Now we can start using the macros included above to define the actual youbot -->
   <!-- The first use of a macro.  This one was defined in base.urdf.xacro above.
@@ -24,5 +24,14 @@
        the origin block defines where the component is w.r.t its parent (in this case the parent
        is the world frame). For more, see http://www.ros.org/wiki/xacro -->
-  <!-- foot for arm-->
+  <xacro:youbot_arm_control
+    name="arm"
+    ec_interface="enx00e04c05e466"
+    ec_cycle_us="1000"
+    ec_timeout_pd_us="500"
+    ec_timeout_mbxrx_us="200"
+    ec_timeout_mbxtx_us="200"
+    diagnostics_cycle_ms="500"
+  />
+  <!-- base for arm-->
   <link name="base_link">
     <inertial>
@@ -36,6 +45,8 @@
     <origin xyz="0.143 0 0.046" rpy="0 0 0" />
   </xacro:youbot_arm>
-  <xacro:youbot_gripper name="gripper" parent="arm_link_5">
-    <origin xyz="0 0 0" rpy="0 0 0" />
-  </xacro:youbot_gripper>
+  <!--
+    <xacro:youbot_gripper name="gripper" parent="arm_link_5">
+      <origin xyz="0 0 0" rpy="0 0 0" />
+    </xacro:youbot_gripper>
+  -->
 </robot>

File: description/urdf/youbot_arm/arm.urdf.xacro (robot description, xacro)
@@ -4,7 +4,7 @@
         xmlns:interface="http://playerstage.sourceforge.net/gazebo/xmlschema/#interface"
         xmlns:xacro="http://www.ros.org/wiki/xacro/#interface">
-	<xacro:include filename="$(find youbot_description)/urdf/youbot_arm/arm.gazebo.xacro" />
-	<xacro:include filename="$(find youbot_description)/urdf/youbot_arm/arm.transmission.xacro" />
-	<xacro:include filename="$(find youbot_description)/urdf/youbot_arm/limits.urdf.xacro" />
+	<!-- <xacro:include filename="$(find youbot_ros2)/description/urdf/youbot_arm/arm.gazebo.xacro" /> -->
+	<!-- <xacro:include filename="$(find youbot_ros2)/description/urdf/youbot_arm/arm.transmission.xacro" /> -->
+	<xacro:include filename="$(find youbot_ros2)/description/urdf/youbot_arm/arm.constants_limits.urdf.xacro" />
 	<xacro:macro name="youbot_arm" params="parent name *origin">
 		<!-- joint between base_link and arm_0_link -->
@@ -24,5 +24,5 @@
 				<origin xyz="0 0 0" rpy="0 0 0" />
 				<geometry>
-					<mesh filename="package://youbot_description/meshes/youbot_arm/arm0.dae" />
+					<mesh filename="package://youbot_ros2/description/meshes/youbot_arm/arm0.dae" />
 				</geometry>
 				<material name="youBot/DarkGrey" />
@@ -32,5 +32,5 @@
 				<origin xyz="0 0 0" rpy="0 0 0"/>
 				<geometry>
-					<mesh filename="package://youbot_description/meshes/youbot_arm/arm0_convex.dae" />
+					<mesh filename="package://youbot_ros2/description/meshes/youbot_arm/arm0_convex.dae" />
 					<!--<cylinder length="0.078" radius="0.093"/>-->
 				</geometry>
@@ -63,5 +63,5 @@
 				<origin xyz="0 0 0" rpy="0 0 0" />
 				<geometry>
-					<mesh filename="package://youbot_description/meshes/youbot_arm/arm1.dae" />
+					<mesh filename="package://youbot_ros2/description/meshes/youbot_arm/arm1.dae" />
 				</geometry>
 				<material name="youBot/Orange" />
@@ -71,5 +71,5 @@
 				<origin xyz="0 0 0" rpy="0 0 0" />
 				<geometry>
-					<mesh filename="package://youbot_description/meshes/youbot_arm/arm1_convex.dae" />
+					<mesh filename="package://youbot_ros2/description/meshes/youbot_arm/arm1_convex.dae" />
 					<!--<cylinder length="0.102" radius="0.080"/>-->
 				</geometry>
@@ -95,5 +95,5 @@
 			<origin xyz="0 -0.032 0.078" rpy="0 0 0" />
 				<geometry>
-					<mesh filename="package://youbot_description/meshes/youbot_arm/arm2.dae" />
+					<mesh filename="package://youbot_ros2/description/meshes/youbot_arm/arm2.dae" />
 				</geometry>
 			</visual>
@@ -102,5 +102,5 @@
 				<origin xyz="0 -0.032 0.078" rpy="0 0 0" />
 				<geometry>
-					<mesh filename="package://youbot_description/meshes/youbot_arm/arm2_convex.dae" />
+					<mesh filename="package://youbot_ros2/description/meshes/youbot_arm/arm2_convex.dae" />
 					<!--<box size="0.074 0.082 0.222"/>-->
 				</geometry>
@@ -134,5 +134,5 @@
 				<origin xyz="0.000 0.028 0.079" rpy="0 0 0" />
 				<geometry>
-					<mesh filename="package://youbot_description/meshes/youbot_arm/arm3.dae" />
+					<mesh filename="package://youbot_ros2/description/meshes/youbot_arm/arm3.dae" />
 				</geometry>
 				<material name="youBot/Orange" />
@@ -142,5 +142,5 @@
 				<origin xyz="0.000 0.028 0.079" rpy="0 0 0" />
 				<geometry>
-					<mesh filename="package://youbot_description/meshes/youbot_arm/arm3_convex.dae" />
+					<mesh filename="package://youbot_ros2/description/meshes/youbot_arm/arm3_convex.dae" />
 					<!--<box size="0.064 0.054 0.192"/>-->
 				</geometry>
@@ -166,5 +166,5 @@
 				<origin xyz="0 -0.010 0.029" rpy="0 0 0"/>
 				<geometry>
-					<mesh filename="package://youbot_description/meshes/youbot_arm/arm4.dae" />
+					<mesh filename="package://youbot_ros2/description/meshes/youbot_arm/arm4.dae" />
 				</geometry>
 				<material name="youBot/Orange" />
@@ -174,5 +174,5 @@
 				<origin xyz="0 -0.010 0.029" rpy="0 0 0"/>
 				<geometry>
-					<mesh filename="package://youbot_description/meshes/youbot_arm/arm4_convex.dae" />
+					<mesh filename="package://youbot_ros2/description/meshes/youbot_arm/arm4_convex.dae" />
 					<!--<box size="0.058 0.100 0.118"/>-->
 				</geometry>
@@ -198,5 +198,5 @@
 				<origin xyz="0.003 0 -0.034" rpy="0 0 0" />
 				<geometry>
-					<mesh filename="package://youbot_description/meshes/youbot_arm/arm5.dae" />
+					<mesh filename="package://youbot_ros2/description/meshes/youbot_arm/arm5.dae" />
 				</geometry>
 				<material name="youBot/DarkGrey" />
@@ -205,5 +205,5 @@
 				<origin xyz="0.003 0 -0.034" rpy="0 0 0" />
 				<geometry>
-					<mesh filename="package://youbot_description/meshes/youbot_arm/arm5_convex.dae" />
+					<mesh filename="package://youbot_ros2/description/meshes/youbot_arm/arm5_convex.dae" />
 					<!--<box size="0.054 0.096 0.030"/>-->
 				</geometry>
@@ -211,6 +211,9 @@
 		</link>
 		<!-- extensions -->
-		<xacro:youbot_arm_gazebo name="${name}" />
-		<xacro:youbot_arm_transmission name="${name}" />
+		<!-- both likely only needed for gazebo simulation -->
+		<!--
+			<xacro:youbot_arm_gazebo name="${name}" />
+			<xacro:youbot_arm_transmission name="${name}" />
+		-->
 	</xacro:macro>
 </robot>
